File: 6809RetroBB/ram_rom.kicad_sch (KiCad schematic)
At the start: 30 parts

Commit message: Minor comments
Parts:
- removed U?: 74LS00, symbol 74xx:74LS00
- added U?: 74LS00, symbol 74xx:74LS00
- added U?: 74LS02, symbol 74xx:74LS02
Connections:
- net +5V: now also U?.1, U?.1, U?.2, U?.2; no longer U?.10, U?.13, U?.4, U?.9
- net E ACIA,PIA: now also U?.3; no longer U?.8
- net E LCD,LED: now also U?.3; no longer U?.6
- net E RAM,ROM: now also U?.3; no longer U?.11
- net R/~{W}: now also U?.1, U?.2, U?.2; no longer U?.4, U?.5, U?.6
- net at U?.11 (Cp): now also U?.1; no longer U?.4
- net at U?.15 (O0): now also U?.2; no longer U?.5
- net at U?.1, U?.2, U?.22 (~{OE}): now also U?.3; no longer U?.6
- net at U?.12 (O3): now also U?.2; no longer U?.10
- net at U?.13 (O2): now also U?.4; no longer U?.12
- net at U?.14 (O1): now also U?.5; no longer U?.13
- new net: U?.1, U?.3
- new net: U?.1, U?.1, U?.2, U?.34 (E)
- new net: U?.1, U?.20 (~{CS}), U?.6
- new net: U?.2, U?.2, U?.3
- new net Q: U?.1, U?.2
- new net ~{Q}: U?.3, U?.3
Other:
- note removed: "Gating with E Clock Stablilizes R/~{W} Effectively syncrohizes."
